File: Board/EmergencyWake.sch (KiCad schematic (older format))
At the start: 103 parts, among them J1 Barrel_Jack_Switch, J2 Micro_SD_Card_Det, J3 Conn_01x04, J4 Conn_01x02, J5 Conn_01x03, J6 Conn_01x03, J7 Conn_01x02, J8 Conn_01x04, J9 Conn_01x04, Q2 AO3400A, SW1 SW_Push, SW2 SW_DPDT_x2, SW3 SW_Push, U2 STM32F103VETx, U3 M24C02-WMN, U4 LM4670, Y1 32,768

Commit message: [Board] Wired all signals to STM32
Parts:
- removed J1: Barrel_Jack_Switch, Connector_BarrelJack:BarrelJack_CUI_PJ-102AH_Horizontal, symbol Connector:Barrel_Jack_Switch
- added J?: USB_C_Plug_USB2.0, Wuerth:632723300011, symbol Connector:USB_C_Plug_USB2.0
- added R?: 100k, Resistor_SMD:R_0402_1005Metric, symbol Device:R
- added R?: 1.5k, Resistor_SMD:R_0402_1005Metric, symbol Device:R
- added R? (x2): 390, Resistor_SMD:R_0603_1608Metric, symbol Device:R
- added R? (x2): 10k, Resistor_SMD:R_0402_1005Metric, symbol Device:R
- added TP? (x2): TestPoint, TestPoint:TestPoint_Loop_D1.80mm_Drill1.0mm_Beaded, symbol Connector:TestPoint
- added U? (x2): EL357N-G, Package_SO:SOP-4_3.8x4.1mm_P2.54mm, symbol Isolator:TLP785
- BT1: Conrad (none) -> 1009388 - 62
- J2: Conrad (none) -> 1308329 - 62
- R?: footprint (none) -> Wuerth:561070332057
Connections:
- net labels added: SD_CK, SD_CMD, SD_CS, SD_D0, SD_MISO, SD_MOSI, SD_SCK, USB_DM, USB_DP, Vdrive
- wire segments 432 -> 509
- no-connect marks 20 -> 57
Other:
- note added: "V_drive is 3.3 V\nabove -VDC"
- note removed: "V_fil is 3.3 V\nabove -VDC"
- moved on the sheet: BT1, C1, C10, C16, C17, C18, C19, C6, C?, D1, D?, DISP1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

Commit message: [Board] Cleaned up schematic sections
Parts:
- added JP? (x3): SolderJumper_3_Open, Jumper:SolderJumper-3_P1.3mm_Open_RoundedPad1.0x1.5mm_NumberLabels, symbol Jumper:SolderJumper_3_Open
Connections:
- net SD_D3_CS is gone; now on net SD_CS: J2.2 (DAT3/CD), R8.2
- net SD_CK: now also JP?.1 (A)
- net SD_CLK: now also JP?.2 (C)
- net SD_CMD: now also JP?.1 (A)
- net SD_CMD_MOSI: now also JP?.2 (C)
- net SD_D0: now also JP?.1 (A)
- net SD_D0_MISO: now also JP?.2 (C)
- net SD_MISO: now also JP?.3 (B)
- net SD_MOSI: now also JP?.3 (B)
- net SD_SCK: now also JP?.3 (B)
- net SEG_L: now reaches DISP1.9 (l), U?.26 (SG12/GR11)
- net SD_D1: no longer names the net of J2.8 (DAT1), R15.2
- net SD_D2: no longer names the net of J2.1 (DAT2), R7.2
Other:
- moved on the sheet: C11, C12, C13, C2, C3, C4, C5, C7, C8, C9, C?, D?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

Commit message: [Board] Switched some pins around
Parts:
- removed R?: 10k, Resistor_SMD:R_0402_1005Metric, symbol Device:R
- added Q2: AO3401A, Package_TO_SOT_SMD:SOT-23, symbol Device:Q_PMOS_GSD
- added R17: 100k, Resistor_SMD:R_0402_1005Metric, symbol Device:R
- added R23: 20k, Resistor_SMD:R_0603_1608Metric, symbol Device:R
- added R37: 10k, Resistor_SMD:R_0603_1608Metric, symbol Device:R
- added TP10: -17V, TestPoint:TestPoint_Loop_D1.80mm_Drill1.0mm_Beaded, symbol Connector:TestPoint
- added TP5: DCDC in, TestPoint:TestPoint_Loop_D1.80mm_Drill1.0mm_Beaded, symbol Connector:TestPoint
- added TP8: -20V, TestPoint:TestPoint_Loop_D1.80mm_Drill1.0mm_Beaded, symbol Connector:TestPoint
- added TP9: LDR, TestPoint:TestPoint_Loop_D1.80mm_Drill1.0mm_Beaded, symbol Connector:TestPoint
- D1, D2, D3, D4: renamed from D?; value LED -> white
- R25: renamed from R?; footprint (none) -> Resistor_SMD:R_0603_1608Metric
- R38, R39: renamed from R?; footprint Resistor_SMD:R_0402_1005Metric -> Resistor_SMD:R_0603_1608Metric; LCSC C25744 -> C25804
- TP1: renamed from TP?; value TestPoint -> 5V in
- TP2: renamed from TP?; value TestPoint -> GND in
- TP3: renamed from TP2; value TestPoint -> 5V
- TP4: value TestPoint -> 3V
- TP6: renamed from TP5; value TestPoint -> GND
- TP7: renamed from TP6; value TestPoint -> Audio
- gave numbers to parts that had none: 32
- renumbered C2 to C1, C12 to C10, C13 to C12, C10 to C13, C14 to C15, C15 to C17, C16 to C19, C4 to C2, C17 to C20, C1 to C21, C19 to C22, C18 to C24, C20 to C26, C22 to C27, C23 to C28, C21 to C29, C24 to C30, C25 to C31, C26 to C32, C5 to C4, C7 to C5, C8 to C6, C9 to C7, C11 to C8, C6 to C9, D1 to D5, J6 to J3, J7 to J4, J9 to J6, J4 to J7, J3 to J8, J8 to J9, JP1 to JP4, Q2 to Q1, R5 to R1, R8 to R10, R15 to R16, R16 to R21, R17 to R22, R1 to R24, R19 to R26, R20 to R27, R21 to R28, R22 to R29, R18 to R30, R23 to R31, R24 to R32, R25 to R33, R26 to R34, R27 to R40, R6 to R8, R7 to R9, TP7 to TP11, U3 to U1, U2 to U4, U4 to U5
Connections:
- net +5V: now also Q2.2 (S), R17.1; no longer R18.1, U3.6 (Vin)
- net -VDC: now also TP8.1
- net EEPROM_SCL: now also U4.92 (PB6); no longer U4.95 (PB8)
- net EEPROM_SDA: now also U4.93 (PB7); no longer U4.96 (PB9)
- net GND: now also R24.2
- net LED1: now also U4.15 (PC0); no longer U4.85 (PD4)
- net LED2: now also U4.16 (PC1); no longer U4.86 (PD5)
- net LED3: now also U4.17 (PC2); no longer U4.87 (PD6)
- net LED4: now also U4.18 (PC3); no longer U4.88 (PD7)
- net SD_CS: now also U4.77 (PA15); no longer U4.33 (PC4)
- net SD_DET: now also U4.87 (PD6); no longer U4.34 (PC5)
- net SD_EN: now also U4.86 (PD5); no longer U4.35 (PB0)
- net SD_MISO: now also U4.90 (PB4); no longer U4.31 (PA6)
- net SD_MOSI: now also U4.91 (PB5); no longer U4.32 (PA7)
- net SD_SCK: now also U4.89 (PB3); no longer U4.30 (PA5)
- net VCC: now also R23.1, R37.1
- net Vdrive: now also TP10.1
- net at R24.1: now also U4.31 (PA6), R23.2, TP9.1
- net at J8.1 (Pin_1): now also R37.2
- net DCDC_EN: now reaches U4.62 (PD15)
- net DCDC_EN: now also Q2.1 (G), R17.2
- net SD_CLK renamed SD_CK_SCK
- new net: Q2.3 (D), R18.1, TP5.1, U3.6 (Vin)
- no-connect marks 57 -> 55
Other:
- note added: "Negative supply for VFD\nSet to -19.63 V"
- note removed: "Negative supply for VFD\nSet to 19.63 V"
- moved on the sheet: C14, C16, C28, C29, R24

Commit message: [Board] Placed a lot of components!
Parts:
- SW1: renamed from SW2; footprint Switch:SlidingSwitch_6pin -> Wuerth:452404020202; Würth (none) -> 452404020202
- SW2: renamed from SW1; footprint (none) -> Wuerth:436351045816; Würth (none) -> 436351045816
- SW3, SW4: footprint (none) -> Wuerth:436351045816; Würth (none) -> 436351045816
Connections:
- net +3V0: now also D5.2 (A); no longer SW1.5 (B)
- net VCC: now also SW1.4 (A); no longer D5.1 (K)
- new net: D5.1 (K), SW1.5 (B)
- no-connect marks 55 -> 57
Other:
- moved on the sheet: D5, SW1B, TP4
Changed lines of the file:
@@
 U 1 1 5E2C7D9C
 P 9400 8600
-F 0 "C21" H 9515 8646 50  0000 L CNN
-F 1 "6p" H 9515 8555 50  0000 L CNN
+F 0 "C21" H 9150 8650 50  0000 L CNN
+F 1 "6p" H 9200 8550 50  0000 L CNN
 F 2 "Capacitor_SMD:C_0402_1005Metric" H 9438 8450 50  0001 C CNN
 F 3 "~" H 9400 8600 50  0001 C CNN
@@
 L Device:D_Schottky D5
 U 1 1 5E2D4271
-P 5350 1150
-F 0 "D5" H 5350 1366 50  0000 C CNN
-F 1 "SS54" H 5350 1275 50  0000 C CNN
-F 2 "Diode_SMD:D_SMA" H 5350 1150 50  0001 C CNN
-F 3 "~" H 5350 1150 50  0001 C CNN
-F 4 "C22452" H 5350 1150 50  0001 C CNN "LCSC"
-	1    5350 1150
+P 5900 1150
+F 0 "D5" H 5900 1366 50  0000 C CNN
+F 1 "SS54" H 5900 1275 50  0000 C CNN
+F 2 "Diode_SMD:D_SMA" H 5900 1150 50  0001 C CNN
+F 3 "~" H 5900 1150 50  0001 C CNN
+F 4 "C22452" H 5900 1150 50  0001 C CNN "LCSC"
+	1    5900 1150
 	1    0    0    1
 $EndComp
@@
 	4500 1150 4650 1150
 Wire Wire Line
-	4650 1150 4650 950
+	4650 1150 4650 1050
 Wire Wire Line
 	4650 1450 4650 1500
@@
 	6600 1150 6050 1150
 Connection ~ 6600 1150
-Wire Wire Line
-	4650 1150 4800 1150
 $Comp
 L Connector_Generic:Conn_01x03 J5
@@
 	3100 4800 3400 4800
 $Comp
-L Switch:SW_Push SW1
-U 1 1 5E32DA7D
-P 1100 9050
-F 0 "SW1" H 1100 9335 50  0000 C CNN
-F 1 "SW_Push" H 1100 9244 50  0000 C CNN
-F 2 "" H 1100 9250 50  0001 C CNN
-F 3 "~" H 1100 9250 50  0001 C CNN
-	1    1100 9050
-	1    0    0    -1
-$EndComp
-$Comp
-L Switch:SW_Push SW3
-U 1 1 5E32E356
-P 2800 9050
-F 0 "SW3" H 2800 9335 50  0000 C CNN
-F 1 "SW_Push" H 2800 9244 50  0000 C CNN
-F 2 "" H 2800 9250 50  0001 C CNN
-F 3 "~" H 2800 9250 50  0001 C CNN
-	1    2800 9050
-	1    0    0    -1
-$EndComp
-$Comp
 L power:GND #PWR03
 U 1 1 5E32E7FE
@@
 L Connector:TestPoint TP4
 U 1 1 5EB86E6F
-P 4800 1150
-F 0 "TP4" H 4858 1268 50  0000 L CNN
-F 1 "3V" H 4858 1177 50  0000 L CNN
-F 2 "TestPoint:TestPoint_Loop_D1.80mm_Drill1.0mm_Beaded" H 5000 1150 50  0001 C CNN
-F 3 "~" H 5000 1150 50  0001 C CNN
-	1    4800 1150
+P 4800 1000
+F 0 "TP4" H 4858 1118 50  0000 L CNN
+F 1 "3V" H 4858 1027 50  0000 L CNN
+F 2 "TestPoint:TestPoint_Loop_D1.80mm_Drill1.0mm_Beaded" H 5000 1000 50  0001 C CNN
+F 3 "~" H 5000 1000 50  0001 C CNN
+	1    4800 1000
 	1    0    0    -1
 $EndComp
-Connection ~ 4800 1150
-Wire Wire Line
-	4800 1150 5200 1150
 $Comp
 L Connector:TestPoint TP6
@@
 	14600 7500 14350 7500
 $Comp
-L Switch:SW_DPDT_x2 SW2
+L Switch:SW_DPDT_x2 SW1
 U 1 1 5E4D4D81
 P 2700 950
-F 0 "SW2" H 2700 1235 50  0000 C CNN
+F 0 "SW1" H 2700 1235 50  0000 C CNN
 F 1 "SW_DPDT_x2" H 2700 1144 50  0000 C CNN
-F 2 "Switch:SlidingSwitch_6pin" H 2700 950 50  0001 C CNN
-F 3 "~" H 2700 950 50  0001 C CNN
+F 2 "Wuerth:452404020202" H 2700 950 50  0001 C CNN
+F 3 "https://www.we-online.de/katalog/datasheet/452404020202.pdf" H 2700 950 50  0001 C CNN
+F 4 "452404020202" H 2700 950 50  0001 C CNN "Würth"
 	1    2700 950
 	1    0    0    -1
 $EndComp
 $Comp
-L Switch:SW_DPDT_x2 SW2
+L Switch:SW_DPDT_x2 SW1
 U 2 1 5E4D5E2F
-P 5800 1250
-F 0 "SW2" H 5800 1535 50  0000 C CNN
-F 1 "SW_DPDT_x2" H 5800 1444 50  0000 C CNN
-F 2 "Switch:SlidingSwitch_6pin" H 5800 1250 50  0001 C CNN
-F 3 "~" H 5800 1250 50  0001 C CNN
-	2    5800 1250
+P 5450 1150
+F 0 "SW1" H 5450 1435 50  0000 C CNN
+F 1 "SW_DPDT_x2" H 5450 1344 50  0000 C CNN
+F 2 "Wuerth:452404020202" H 5450 1150 50  0001 C CNN
+F 3 "https://www.we-online.de/katalog/datasheet/452404020202.pdf" H 5450 1150 50  0001 C CNN
+F 4 "452404020202" H 5450 1150 50  0001 C CNN "Würth"
+	2    5450 1150
 	-1   0    0    -1
 $EndComp
@@
 Connection ~ 6600 1500
 Wire Wire Line
-	6050 1150 6050 1250
-Wire Wire Line
-	6050 1250 6000 1250
-Wire Wire Line
 	4650 1500 6600 1500
 $Comp
@@
 Text Label 10500 6850 0    50   ~ 0
 VFD_STB
-Wire Wire Line
-	5500 1150 5600 1150
 NoConn ~ 11150 7100
 NoConn ~ 11150 7300
@@
 Text Label 6100 5400 0    50   ~ 0
 USR_BUT
-$Comp
-L Switch:SW_Push SW4
-U 1 1 5E927342
-P 4000 9050
-F 0 "SW4" H 4000 9335 50  0000 C CNN
-F 1 "SW_Push" H 4000 9244 50  0000 C CNN
-F 2 "" H 4000 9250 50  0001 C CNN
-F 3 "~" H 4000 9250 50  0001 C CNN
-	1    4000 9050
-	1    0    0    -1
-$EndComp
 Text Label 6100 5800 0    50   ~ 0
 DCF_SIG
@@
 	5800 9350 6300 9350
 Connection ~ 6300 9350
+$Comp
+L Switch:SW_Push SW4
+U 1 1 5E927342
+P 4000 9050
+F 0 "SW4" H 4000 9335 50  0000 C CNN
+F 1 "SW_Push" H 4000 9244 50  0000 C CNN
+F 2 "Wuerth:436351045816" H 4000 9250 50  0001 C CNN
+F 3 "~" H 4000 9250 50  0001 C CNN
+F 4 "436351045816" H 4000 9050 50  0001 C CNN "Würth"
+	1    4000 9050
+	1    0    0    -1
+$EndComp
+$Comp
+L Switch:SW_Push SW3
+U 1 1 5E32E356
+P 2800 9050
+F 0 "SW3" H 2800 9335 50  0000 C CNN
+F 1 "SW_Push" H 2800 9244 50  0000 C CNN
+F 2 "Wuerth:436351045816" H 2800 9250 50  0001 C CNN
+F 3 "~" H 2800 9250 50  0001 C CNN
+F 4 "436351045816" H 2800 9050 50  0001 C CNN "Würth"
+	1    2800 9050
+	1    0    0    -1
+$EndComp
+$Comp
+L Switch:SW_Push SW2
+U 1 1 5E32DA7D
+P 1100 9050
+F 0 "SW2" H 1100 9335 50  0000 C CNN
+F 1 "SW_Push" H 1100 9244 50  0000 C CNN
+F 2 "Wuerth:436351045816" H 1100 9250 50  0001 C CNN
+F 3 "~" H 1100 9250 50  0001 C CNN
+F 4 "436351045816" H 1100 9050 50  0001 C CNN "Würth"
+	1    1100 9050
+	1    0    0    -1
+$EndComp
+NoConn ~ 2900 1050
+NoConn ~ 5250 1250
+Wire Wire Line
+	5250 1050 4800 1050
+Connection ~ 4650 1050
+Wire Wire Line
+	4650 1050 4650 950
+Wire Wire Line
+	4800 1000 4800 1050
+Connection ~ 4800 1050
+Wire Wire Line
+	4800 1050 4650 1050
+Wire Wire Line
+	5650 1150 5750 1150
 $EndSCHEMATC

Commit message: [Board] Placed most components, only TPs missing
Parts:
- added R41: 100k, Resistor_SMD:R_0402_1005Metric, symbol Device:R
Connections:
- net AUDIO_EN: now also R41.2
- net VCC: now also R41.1
Changed lines of the file:
@@
 EESchema Schematic File Version 4
+LIBS:EmergencyWake-cache
 EELAYER 30 0
 EELAYER END
@@
 	1    0    0    -1
 $EndComp
-Wire Wire Line
-	9750 1050 7850 1050
 Text Label 7850 1050 0    50   ~ 0
 AUDIO_EN
@@
 Wire Wire Line
 	8800 1250 8750 1250
-Text Notes 8000 1600 0    50   ~ 0
+Text Notes 9400 2100 0    50   ~ 0
 f_C = 1 / (2π*R_i*C_i) (Hz)
 $Comp
@@
 Wire Wire Line
 	5650 1150 5750 1150
+$Comp
+L Device:R R41
+U 1 1 5E442E22
+P 9250 850
+F 0 "R41" H 9320 896 50  0000 L CNN
+F 1 "100k" H 9320 805 50  0000 L CNN
+F 2 "Resistor_SMD:R_0402_1005Metric" V 9180 850 50  0001 C CNN
+F 3 "~" H 9250 850 50  0001 C CNN
+F 4 "C25741" H 9250 850 50  0001 C CNN "LCSC"
+	1    9250 850
+	1    0    0    -1
+$EndComp
+Wire Wire Line
+	9750 1050 9250 1050
+$Comp
+L power:VCC #PWR072
+U 1 1 5E4E85D6
+P 9400 650
+F 0 "#PWR072" H 9400 500 50  0001 C CNN
+F 1 "VCC" H 9417 823 50  0000 C CNN
+F 2 "" H 9400 650 50  0001 C CNN
+F 3 "" H 9400 650 50  0001 C CNN
+	1    9400 650
+	0    1    1    0
+$EndComp
+Wire Wire Line
+	9400 650  9250 650
+Wire Wire Line
+	9250 650  9250 700
+Wire Wire Line
+	9250 1000 9250 1050
+Connection ~ 9250 1050
+Wire Wire Line
+	9250 1050 7850 1050
 $EndSCHEMATC

Commit message: [Board] Changed lever to active high, replaced LDO for filament
Parts:
- removed U6: AMS1117-3.3, Package_TO_SOT_SMD:SOT-223-3_TabPin2, symbol Regulator_Linear:AMS1117-3.3
- added U6: 173950378, Converter_DCDC:Converter_DCDC_RECOM_R-78B-2.0_THT, symbol Regulator_Switching:R-78B1.2-2.0
Connections:
- net -VDC: now also U6.2 (GND)
- net GND: now also R30.2, U6.1 (IN); no longer J4.2 (Pin_2)
- net VCC: now also J4.2 (Pin_2); no longer R30.2
- net Vdrive: now also U6.3 (OUT)
Changed lines of the file:
@@
 EESchema Schematic File Version 4
-LIBS:EmergencyWake-cache
 EELAYER 30 0
 EELAYER END
@@
 $EndComp
 $Comp
-L power:VCC #PWR044
-U 1 1 5E409EAE
-P 11900 850
-F 0 "#PWR044" H 11900 700 50  0001 C CNN
-F 1 "VCC" V 11918 977 50  0000 L CNN
-F 2 "" H 11900 850 50  0001 C CNN
-F 3 "" H 11900 850 50  0001 C CNN
-	1    11900 850
-	0    -1   -1   0
-$EndComp
-$Comp
 L power:GND #PWR060
 U 1 1 5E40A4BA
-P 13700 2500
-F 0 "#PWR060" H 13700 2250 50  0001 C CNN
-F 1 "GND" H 13705 2327 50  0000 C CNN
-F 2 "" H 13700 2500 50  0001 C CNN
-F 3 "" H 13700 2500 50  0001 C CNN
-	1    13700 2500
+P 11900 2400
+F 0 "#PWR060" H 11900 2150 50  0001 C CNN
+F 1 "GND" H 11905 2227 50  0000 C CNN
+F 2 "" H 11900 2400 50  0001 C CNN
+F 3 "" H 11900 2400 50  0001 C CNN
+	1    11900 2400
 	0    1    1    0
 $EndComp
@@
 $EndComp
 $Comp
-L power:VCC #PWR048
-U 1 1 5E63717C
-P 11900 2400
-F 0 "#PWR048" H 11900 2250 50  0001 C CNN
-F 1 "VCC" V 11918 2527 50  0000 L CNN
-F 2 "" H 11900 2400 50  0001 C CNN
-F 3 "" H 11900 2400 50  0001 C CNN
-	1    11900 2400
-	0    -1   -1   0
-$EndComp
-$Comp
 L Device:R R30
 U 1 1 5E637187
@@
 $EndComp
 $Comp
-L power:GND #PWR049
-U 1 1 5E63719C
-P 11900 2800
-F 0 "#PWR049" H 11900 2550 50  0001 C CNN
-F 1 "GND" H 11905 2627 50  0000 C CNN
-F 2 "" H 11900 2800 50  0001 C CNN
-F 3 "" H 11900 2800 50  0001 C CNN
-	1    11900 2800
-	0    1    1    0
-$EndComp
-$Comp
-L power:VCC #PWR046
-U 1 1 5E640E6F
-P 11900 1600
-F 0 "#PWR046" H 11900 1450 50  0001 C CNN
-F 1 "VCC" V 11918 1727 50  0000 L CNN
-F 2 "" H 11900 1600 50  0001 C CNN
-F 3 "" H 11900 1600 50  0001 C CNN
-	1    11900 1600
-	0    -1   -1   0
-$EndComp
-$Comp
 L Device:R R29
 U 1 1 5E640E7A
@@
 	0    -1   -1   0
 $EndComp
-$Comp
-L Regulator_Linear:AMS1117-3.3 U6
-U 1 1 5E4459B5
-P 10450 10150
-F 0 "U6" H 10450 10392 50  0000 C CNN
-F 1 "AMS1117-3.3" H 10450 10301 50  0000 C CNN
-F 2 "Package_TO_SOT_SMD:SOT-223-3_TabPin2" H 10450 10350 50  0001 C CNN
-F 3 "http://www.advanced-monolithic.com/pdf/ds1117.pdf" H 10550 9900 50  0001 C CNN
-F 4 "C6186" H 10450 10150 50  0001 C CNN "LCSC"
-	1    10450 10150
-	1    0    0    -1
-$EndComp
 Wire Wire Line
 	15150 7050 15150 7500
@@
 Wire Notes Line
 	5050 2300 11450 2300
-$Comp
-L power:GND #PWR059
-U 1 1 5E40A111
-P 13700 2150
-F 0 "#PWR059" H 13700 1900 50  0001 C CNN
-F 1 "GND" H 13705 1977 50  0000 C CNN
-F 2 "" H 13700 2150 50  0001 C CNN
-F 3 "" H 13700 2150 50  0001 C CNN
-	1    13700 2150
-	0    1    1    0
-$EndComp
 Wire Wire Line
 	12250 2050 13700 2050
@@
 Wire Wire Line
 	9250 1050 7850 1050
+$Comp
+L power:VCC #PWR044
+U 1 1 5E409EAE
+P 11900 850
+F 0 "#PWR044" H 11900 700 50  0001 C CNN
+F 1 "VCC" V 11918 977 50  0000 L CNN
+F 2 "" H 11900 850 50  0001 C CNN
+F 3 "" H 11900 850 50  0001 C CNN
+	1    11900 850
+	0    -1   -1   0
+$EndComp
+$Comp
+L power:GND #PWR049
+U 1 1 5E63719C
+P 11900 2800
+F 0 "#PWR049" H 11900 2550 50  0001 C CNN
+F 1 "GND" H 11905 2627 50  0000 C CNN
+F 2 "" H 11900 2800 50  0001 C CNN
+F 3 "" H 11900 2800 50  0001 C CNN
+	1    11900 2800
+	0    1    1    0
+$EndComp
+$Comp
+L power:VCC #PWR048
+U 1 1 5E63717C
+P 13700 2500
+F 0 "#PWR048" H 13700 2350 50  0001 C CNN
+F 1 "VCC" V 13718 2627 50  0000 L CNN
+F 2 "" H 13700 2500 50  0001 C CNN
+F 3 "" H 13700 2500 50  0001 C CNN
+	1    13700 2500
+	0    -1   -1   0
+$EndComp
+$Comp
+L power:GND #PWR059
+U 1 1 5E40A111
+P 13700 2150
+F 0 "#PWR059" H 13700 1900 50  0001 C CNN
+F 1 "GND" H 13705 1977 50  0000 C CNN
+F 2 "" H 13700 2150 50  0001 C CNN
+F 3 "" H 13700 2150 50  0001 C CNN
+	1    13700 2150
+	0    1    1    0
+$EndComp
+$Comp
+L power:VCC #PWR046
+U 1 1 5E640E6F
+P 11900 1600
+F 0 "#PWR046" H 11900 1450 50  0001 C CNN
+F 1 "VCC" V 11918 1727 50  0000 L CNN
+F 2 "" H 11900 1600 50  0001 C CNN
+F 3 "" H 11900 1600 50  0001 C CNN
+	1    11900 1600
+	0    -1   -1   0
+$EndComp
+$Comp
+L Regulator_Switching:R-78B1.2-2.0 U6
+U 1 1 5E42AF9F
+P 10450 10150
+F 0 "U6" H 10450 10392 50  0000 C CNN
+F 1 "173950378" H 10450 10301 50  0000 C CNN
+F 2 "Converter_DCDC:Converter_DCDC_RECOM_R-78B-2.0_THT" H 10500 9900 50  0001 L CIN
+F 3 "https://www.we-online.de/katalog/datasheet/173950378.pdf" H 10450 10150 50  0001 C CNN
+F 4 "173950378" H 10450 10150 50  0001 C CNN "Würth"
+	1    10450 10150
+	1    0    0    -1
+$EndComp
 $EndSCHEMATC

Commit message: [Board] Finished moving components to front of board
Parts:
- U5: LCSC (none) -> C131968
Connections:
- net +3V0: now also SW1.5 (B); no longer D5.2 (A)
- net DCF_PON: no longer TP11.1
- net DCF_SIG: now also TP11.1
- net VCC: now also D5.1 (K); no longer SW1.4 (A)
- new net: D5.2 (A), SW1.4 (A)
Other:
- moved on the sheet: D5, SW1B, TP11
Changed lines of the file:
@@
 $EndComp
 $Comp
-L Device:D_Schottky D5
-U 1 1 5E2D4271
-P 5900 1150
-F 0 "D5" H 5900 1366 50  0000 C CNN
-F 1 "SS54" H 5900 1275 50  0000 C CNN
-F 2 "Diode_SMD:D_SMA" H 5900 1150 50  0001 C CNN
-F 3 "~" H 5900 1150 50  0001 C CNN
-F 4 "C22452" H 5900 1150 50  0001 C CNN "LCSC"
-	1    5900 1150
-	1    0    0    1
-$EndComp
-$Comp
 L power:GND #PWR018
 U 1 1 5E2D57EC
@@
 Wire Wire Line
 	3400 1150 3900 1150
-Text Notes 4800 800  0    50   ~ 0
+Text Notes 4800 750  0    50   ~ 0
 cp. https://www.st.com/resource/en/application_note/dm00206898.pdf
 $Comp
@@
 $EndComp
 Wire Wire Line
-	13050 3500 13700 3500
+	13050 3500 13450 3500
 Text Label 13050 3400 0    50   ~ 0
 DCF_PON
@@
 	12050 3200 13700 3200
 Wire Wire Line
-	12400 3400 12500 3400
-Wire Wire Line
 	11550 3500 12950 3500
 $Comp
@@
 L Connector:TestPoint TP11
 U 1 1 5E414D66
-P 12500 3400
-F 0 "TP11" H 12558 3518 50  0000 L CNN
-F 1 "TestPoint" H 12558 3427 50  0000 L CNN
-F 2 "TestPoint:TestPoint_Loop_D1.80mm_Drill1.0mm_Beaded" H 12700 3400 50  0001 C CNN
-F 3 "~" H 12700 3400 50  0001 C CNN
-	1    12500 3400
-	1    0    0    -1
+P 13450 3500
+F 0 "TP11" H 13508 3618 50  0000 L CNN
+F 1 "TestPoint" H 13508 3527 50  0000 L CNN
+F 2 "TestPoint:TestPoint_Loop_D1.80mm_Drill1.0mm_Beaded" H 13650 3500 50  0001 C CNN
+F 3 "~" H 13650 3500 50  0001 C CNN
+	1    13450 3500
+	-1   0    0    1
 $EndComp
-Connection ~ 12500 3400
-Wire Wire Line
-	12500 3400 13700 3400
 Text Notes 15800 7500 1    50   ~ 0
 Grid 3 can either be permanently\nactive be driven together with\nGrid 2 (selectable by solder jumper)
@@
 L Switch:SW_DPDT_x2 SW1
 U 2 1 5E4D5E2F
-P 5450 1150
-F 0 "SW1" H 5450 1435 50  0000 C CNN
-F 1 "SW_DPDT_x2" H 5450 1344 50  0000 C CNN
-F 2 "Wuerth:452404020202" H 5450 1150 50  0001 C CNN
-F 3 "https://www.we-online.de/katalog/datasheet/452404020202.pdf" H 5450 1150 50  0001 C CNN
-F 4 "452404020202" H 5450 1150 50  0001 C CNN "Würth"
-	2    5450 1150
+P 5850 1150
+F 0 "SW1" H 5850 1435 50  0000 C CNN
+F 1 "SW_DPDT_x2" H 5850 1344 50  0000 C CNN
+F 2 "Wuerth:452404020202" H 5850 1150 50  0001 C CNN
+F 3 "https://www.we-online.de/katalog/datasheet/452404020202.pdf" H 5850 1150 50  0001 C CNN
+F 4 "452404020202" H 5850 1150 50  0001 C CNN "Würth"
+	2    5850 1150
 	-1   0    0    -1
 $EndComp
@@
 F 2 "Package_SON:WSON-8-1EP_3x3mm_P0.5mm_EP1.6x2.0mm" H 10200 600 50  0001 C CNN
 F 3 "https://datasheet.lcsc.com/szlcsc/Texas-Instruments-TI-LM4670SD-NOPB_C131968.pdf" H 10100 1900 50  0001 C CNN
+F 4 "C131968" H 10200 1350 50  0001 C CNN "LCSC"
 	1    10200 1350
 	1    0    0    -1
@@
 $EndComp
 NoConn ~ 2900 1050
-NoConn ~ 5250 1250
-Wire Wire Line
-	5250 1050 4800 1050
+NoConn ~ 5650 1250
 Connection ~ 4650 1050
 Wire Wire Line
@@
 Wire Wire Line
 	4800 1050 4650 1050
-Wire Wire Line
-	5650 1150 5750 1150
 $Comp
 L Device:R R41
@@
 	1    0    0    -1
 $EndComp
+Wire Wire Line
+	5450 1050 5650 1050
+Wire Wire Line
+	5150 1050 4800 1050
+$Comp
+L Device:D_Schottky D5
+U 1 1 5E2D4271
+P 5300 1050
+F 0 "D5" H 5300 1266 50  0000 C CNN
+F 1 "SS54" H 5300 1175 50  0000 C CNN
+F 2 "Diode_SMD:D_SMA" H 5300 1050 50  0001 C CNN
+F 3 "~" H 5300 1050 50  0001 C CNN
+F 4 "C22452" H 5300 1050 50  0001 C CNN "LCSC"
+	1    5300 1050
+	1    0    0    -1
+$EndComp
+Connection ~ 13450 3500
+Wire Wire Line
+	13450 3500 13700 3500
+Wire Wire Line
+	12400 3400 13700 3400
 $EndSCHEMATC
